File: eagle/ultrasonic_anemometer_pcb.brd (EAGLE design)
At the start: 100 x 80 mm, 66 parts, among them IC1 7805, IC7 ATMEGA1284, Q1 25Mhz, U1 OPAMP-DUALDIP, U2 OPAMP-DUALDIP

Commit message: Small fixes on Eagle pcb schematic.
Parts:
- renumbered PROGRAMATOR to PROGRAMMER
Changed lines of the file:
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@@
 <attribute name="VALUE" x="78.365" y="61.493" size="1.27" layer="27" ratio="10" rot="R270"/>
 </element>
-<element name="PROGRAMATOR" library="jumper" package="JP5Q" value="" x="5" y="40" rot="R270"/>
+<element name="PROGRAMMER" library="jumper" package="JP5Q" value="" x="5" y="40" rot="R270"/>
 <element name="Q1" library="crystal" package="HC49/S" value="25Mhz" x="15" y="26" rot="R90">
 <attribute name="OC_FARNELL" value="1667008" x="15" y="26" size="1.778" layer="27" rot="R90" display="off"/>
@@
 <contactref element="IC7" pad="11"/>
 <contactref element="C14" pad="2"/>
-<contactref element="PROGRAMATOR" pad="1"/>
-<contactref element="PROGRAMATOR" pad="7"/>
-<contactref element="PROGRAMATOR" pad="5"/>
-<contactref element="PROGRAMATOR" pad="3"/>
+<contactref element="PROGRAMMER" pad="1"/>
+<contactref element="PROGRAMMER" pad="7"/>
+<contactref element="PROGRAMMER" pad="5"/>
+<contactref element="PROGRAMMER" pad="3"/>
 <contactref element="C6" pad="1"/>
 <contactref element="C5" pad="1"/>
@@
 <contactref element="R1" pad="2"/>
 <contactref element="IC7" pad="9"/>
-<contactref element="PROGRAMATOR" pad="6"/>
+<contactref element="PROGRAMMER" pad="6"/>
 <wire x1="6.9088" y1="40.64" x2="10.9728" y2="40.64" width="0.4064" layer="1"/>
 <wire x1="6.5024" y1="40.2336" x2="6.9088" y2="40.64" width="0.4064" layer="1"/>
@@
 <signal name="MOSI">
 <contactref element="IC7" pad="6"/>
-<contactref element="PROGRAMATOR" pad="10"/>
+<contactref element="PROGRAMMER" pad="10"/>
 <wire x1="17.4752" y1="45.1104" x2="20.32" y2="45.1104" width="0.4064" layer="16"/>
 <wire x1="7.3152" y1="34.9504" x2="17.4752" y2="45.1104" width="0.4064" layer="16"/>
@@
 <signal name="MISO">
 <contactref element="ADC" pad="6"/>
-<contactref element="PROGRAMATOR" pad="2"/>
+<contactref element="PROGRAMMER" pad="2"/>
 <contactref element="IC7" pad="7"/>
 <wire x1="19.5072" y1="42.672" x2="20.32" y2="42.672" width="0.4064" layer="1"/>
@@
 <signal name="SCK">
 <contactref element="IC7" pad="8"/>
-<contactref element="PROGRAMATOR" pad="4"/>
+<contactref element="PROGRAMMER" pad="4"/>
 <contactref element="ADC" pad="7"/>
 <wire x1="17.4752" y1="40.2336" x2="20.32" y2="40.2336" width="0.4064" layer="16"/>
