File: eagle/ultrasonic_anemometer_pcb.sch (EAGLE design)
At the start: 72 parts, among them IC1 7805, IC7 ATMEGA1284, Q1 25Mhz, U1 OPAMP-DUALDIP, U2 OPAMP-DUALDIP

Commit message: Small fixes on Eagle pcb schematic.
Parts:
- renumbered PROGRAMATOR to PROGRAMMER
Changed lines of the file:
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@@
 <part name="GND3" library="supply1" deviceset="GND" device="" value="DGND"/>
 <part name="P+3" library="supply1" deviceset="VCC" device="" value="+5V"/>
-<part name="PROGRAMATOR" library="jumper" deviceset="JP5Q" device=""/>
+<part name="PROGRAMMER" library="jumper" deviceset="JP5Q" device=""/>
 <part name="GND4" library="supply1" deviceset="GND" device="" value="DGND"/>
 <part name="Q1" library="crystal" deviceset="CRYSTAL" device="HC49S" value="25Mhz"/>
@@
 <attribute name="VALUE" x="-45.72" y="15.24" size="1.778" layer="96"/>
 </instance>
-<instance part="PROGRAMATOR" gate="B" x="53.34" y="-116.84" smashed="yes" rot="R270">
+<instance part="PROGRAMMER" gate="B" x="53.34" y="-116.84" smashed="yes" rot="R270">
 <attribute name="VALUE" x="48.26" y="-126.365" size="1.778" layer="96"/>
 </instance>
@@
 </segment>
 <segment>
-<pinref part="PROGRAMATOR" gate="B" pin="1"/>
+<pinref part="PROGRAMMER" gate="B" pin="1"/>
 <wire x1="45.72" y1="-111.76" x2="43.18" y2="-111.76" width="0.1524" layer="91"/>
-<pinref part="PROGRAMATOR" gate="B" pin="7"/>
+<pinref part="PROGRAMMER" gate="B" pin="7"/>
 <wire x1="45.72" y1="-119.38" x2="43.18" y2="-119.38" width="0.1524" layer="91"/>
 <wire x1="43.18" y1="-119.38" x2="43.18" y2="-116.84" width="0.1524" layer="91"/>
-<pinref part="PROGRAMATOR" gate="B" pin="5"/>
+<pinref part="PROGRAMMER" gate="B" pin="5"/>
 <wire x1="43.18" y1="-116.84" x2="45.72" y2="-116.84" width="0.1524" layer="91"/>
-<pinref part="PROGRAMATOR" gate="B" pin="3"/>
+<pinref part="PROGRAMMER" gate="B" pin="3"/>
 <wire x1="45.72" y1="-114.3" x2="43.18" y2="-114.3" width="0.1524" layer="91"/>
 <wire x1="43.18" y1="-114.3" x2="43.18" y2="-116.84" width="0.1524" layer="91"/>
@@
 </segment>
 <segment>
-<pinref part="PROGRAMATOR" gate="B" pin="6"/>
+<pinref part="PROGRAMMER" gate="B" pin="6"/>
 <wire x1="60.96" y1="-116.84" x2="63.5" y2="-116.84" width="0.1524" layer="91"/>
 <label x="63.5" y="-116.84" size="1.27" layer="95" xref="yes"/>
@@
 </segment>
 <segment>
-<pinref part="PROGRAMATOR" gate="B" pin="10"/>
+<pinref part="PROGRAMMER" gate="B" pin="10"/>
 <wire x1="60.96" y1="-121.92" x2="63.5" y2="-121.92" width="0.1524" layer="91"/>
 <label x="63.5" y="-121.92" size="1.27" layer="95" xref="yes"/>
@@
 </segment>
 <segment>
-<pinref part="PROGRAMATOR" gate="B" pin="2"/>
+<pinref part="PROGRAMMER" gate="B" pin="2"/>
 <wire x1="60.96" y1="-111.76" x2="63.5" y2="-111.76" width="0.1524" layer="91"/>
 <label x="63.5" y="-111.76" size="1.27" layer="95" xref="yes"/>
@@
 </segment>
 <segment>
-<pinref part="PROGRAMATOR" gate="B" pin="4"/>
+<pinref part="PROGRAMMER" gate="B" pin="4"/>
 <wire x1="60.96" y1="-114.3" x2="63.5" y2="-114.3" width="0.1524" layer="91"/>
 <label x="63.5" y="-114.3" size="1.27" layer="95" xref="yes"/>
